File: SIM7080.kicad_pcb (KiCad board)
At the start: 4 copper layers, 38.5 x 47 mm, 55 parts, among them J1 LTE Antenna, J2 GNSS Antenna, J3 USB_B_Micro, J4 SIM_Card, J5 JST PH, J6 Conn_01x10_Male, Q1 FDN340P, Q2 DTC143Z, Q3 DTC143Z, Q4 DTC143Z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

Commit message: ok
Other:
- net class Default removed
